File: PCB/Crazy-75/Crazy-75.kicad_pcb (KiCad board)
At the start: 2 copper layers, 3.6 x 3.3 mm, 330 parts, among them SW1 SW_Push, SW10 SW_Push, SW11 SW_Push, SW12 SW_Push, SW13 SW_Push, SW14 SW_Push, SW15 SW_Push, SW16 SW_Push, SW17 SW_Push, SW18 SW_Push, SW19 SW_Push, SW2 SW_Push, SW20 SW_Push, SW21 SW_Push, SW22 SW_Push, SW23 SW_Push, SW24 SW_Push, SW25 SW_Push, SW26 SW_Push, SW27 SW_Push, SW28 SW_Push, SW29 SW_Push, SW3 SW_Push, SW30 SW_Push, SW31 SW_Push, SW32 SW_Push, SW33 SW_Push, SW34 SW_Push, SW35 SW_Push, SW36 SW_Push, SW37 SW_Push, SW38 SW_Push, SW39 SW_Push, SW4 SW_Push, SW40 SW_Push, SW41 SW_Push, SW42 SW_Push, SW43 SW_Push, SW44 SW_Push, SW45 SW_Push, SW46 SW_Push, SW47 SW_Push, SW48 SW_Push, SW49 SW_Push, SW5 SW_Push, SW50 SW_Push, SW51 SW_Push, SW52 SW_Push, SW53 SW_Push, SW54 SW_Push, SW55 SW_Push, SW56 SW_Push, SW57 SW_Push, SW58 SW_Push, SW59 SW_Push, SW6 SW_Push, SW60 SW_Push, SW61 SW_Push, SW62 SW_Push, SW63 SW_Push, SW64 SW_Push, SW65 SW_Push, SW66 SW_Push, SW67 SW_Push, SW68 SW_Push, SW69 SW_Push, SW7 SW_Push, SW70 SW_Push, SW71 SW_Push, SW72 SW_Push, SW73 SW_Push, SW74 SW_Push, SW75 SW_Push, SW76 SW_Push, SW77 SW_Push, SW78 SW_Push, SW79 SW_Push, SW8 SW_Push, SW80 SW_Push, SW9 SW_Push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

Commit message: 11.09.2026 - PCB design and schematics changes
Parts:
- removed A1: RaspberryPi_Pico, Module:RaspberryPi_Pico_Common_SMD
- removed the C63 at (103.6, -91.5)
- removed D58: 1N4148, Diode_THT:D_DO-35_SOD27_P7.62mm_Horizontal
- removed LED58: SK6812MINI-E, PCM_marbastlib-mx:LED_MX_6028R
- removed SW58: SW_Push, PCM_marbastlib-mx:SW_MX_HS_CPG151101S11_1u
- added C81: 100nF, Capacitor_SMD:C_0805_2012Metric, F.Cu at (95.0, -77.5)
- added C82: 100nF, Capacitor_SMD:C_0805_2012Metric, F.Cu at (155.5, -77.5)
- added LED81: SK6812MINI-E, PCM_marbastlib-mx:LED_MX_6028R, F.Cu at (88.3, -77.4)
- added LED82: SK6812MINI-E, PCM_marbastlib-mx:LED_MX_6028R, F.Cu at (162.5, -77.4)
- added U2: ~, pro_micro_rp2040:pro_micro_rp2040, F.Cu at (283.2, -159.3)
- moved U1 613.7 mm to (298.1, -95.5)
- moved C83 608.6 mm to (293.0, -97.5), turned to 180 degrees
- moved R1 604.4 mm to (293.1, -93.5), turned to 180 degrees
- moved C57 220.2 mm to (265.3, -115.6), turned to -90 degrees
- moved C43 217.8 mm to (272.4, -134.6), turned to -90 degrees
- moved C61 195.9 mm to (72.4, -96.5), turned to -90 degrees
- moved C44 186.6 mm to (299.6, -104.3), turned to -90 degrees
- moved C46 183.6 mm to (43.8, -115.6), turned to -90 degrees
- moved C60 164.6 mm to (53.4, -96.5), turned to -90 degrees
- moved C45 152.7 mm to (17.6, -115.6), turned to -90 degrees
- moved C52 147.5 mm to (158.1, -115.6), turned to -90 degrees
- moved C59 138.4 mm to (22.4, -96.5), turned to -90 degrees
- moved C66 127.2 mm to (167.7, -96.5), turned to -90 degrees
- moved C67 121.4 mm to (186.7, -96.5), turned to -90 degrees
- moved C51 103.5 mm to (139.1, -115.6), turned to -90 degrees
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- renumbered C44 to C42, C47 to C43, C50 to C44, C53 to C45, C56 to C46, C59 to C47, C62 to C48, C65 to C49, C68 to C50, C42 to C51, C45 to C52, C48 to C53, C51 to C54, C54 to C55, C57 to C56, C60 to C57, C66 to C59, C69 to C60, C43 to C61, C46 to C62, C49 to C63, C52 to C64, C55 to C65, C58 to C66, C61 to C67, C64 to C68, C67 to C69, C81 to C83
Connections:
- LED59 pad 3: Net-(LED58-DOUT) -> Net-(LED57-DOUT)
- LED80 pad 2: unconnected-(LED80-DOUT-Pad2) -> Net-(LED80-DOUT)

Commit message: 13.09.2026 - PCB Mechanical Checks & 3D Validation
Continued working on the physical PCB layout and checking whether the component arrangement would actually work mechanically.
Parts:
- LED1, LED10, LED11, LED12, LED13, LED14, LED15, LED16, LED17, LED18, LED19, LED2, LED20, LED21, LED22, LED23, LED24, LED25, LED26, LED27, LED28, LED29, LED3, LED30, LED31, LED32, LED33, LED34, LED35, LED36, LED37, LED38, LED39, LED4, LED40, LED41, LED42, LED43, LED44, LED45, LED46, LED47, LED48, LED49, LED5, LED50, LED51, LED52, LED53, LED54, LED55, LED56, LED57, LED59, LED6, LED60, LED61, LED62, LED63, LED64, LED65, LED66, LED67, LED68, LED69, LED7, LED70, LED71, LED72, LED73, LED74, LED75, LED76, LED77, LED78, LED79, LED8, LED80, LED81, LED82, LED9, SW1, SW10, SW11, SW12, SW13, SW14, SW15, SW16, SW17, SW18, SW19, SW2, SW20, SW21, SW22, SW23, SW24, SW25, SW26, SW27, SW28, SW29, SW3, SW30, SW31, SW32, SW33, SW34, SW35, SW36, SW37, SW38, SW39, SW4, SW40, SW41, SW42, SW43, SW44, SW45, SW46, SW47, SW48, SW49, SW5, SW50, SW51, SW52, SW53, SW54, SW55, SW56, SW57, SW59, SW6, SW60, SW61, SW62, SW63, SW64, SW65, SW66, SW67, SW68, SW69, SW7, SW70, SW71, SW72, SW73, SW74, SW75, SW76, SW77, SW78, SW79, SW8, SW80, SW9: moved to B.Cu
- moved D80 24.6 mm to (301.0, -90.6), turned to -90 degrees
- moved D72 22.5 mm to (-4.00, -97.3), turned to -90 degrees
- moved D59 18.8 mm to (16.3, -111.0), turned to 180 degrees
- moved D28 18.7 mm to (261.3, -168.2), turned to 180 degrees
- moved D30 18.6 mm to (8.57, -149.1), turned to 180 degrees
- moved D34 18.6 mm to (89.5, -149.1), turned to 180 degrees
- moved D35 18.6 mm to (108.6, -149.1), turned to 180 degrees
- moved D38 18.6 mm to (165.7, -149.1), turned to 180 degrees
- moved D31 18.6 mm to (32.4, -149.1), turned to 180 degrees
- moved D32 18.6 mm to (51.4, -149.1), turned to 180 degrees
- moved D33 18.6 mm to (70.5, -149.1), turned to 180 degrees
- moved D36 18.6 mm to (127.6, -149.1), turned to 180 degrees
- moved D37 18.6 mm to (146.7, -149.1), turned to 180 degrees
- moved D39 18.6 mm to (184.8, -149.1), turned to 180 degrees
- moved D41 18.6 mm to (222.9, -149.1), turned to 180 degrees
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Connections:
- U2 pad 13: /COL14 -> unconnected-(U2-GP13-Pad13)
- U2 pad 28: unconnected-(U2-GP28-Pad28) -> /COL14
Other:
- board size 3.6 x 3.3 mm -> 314 x 125.5 mm

Commit message: 14.09.2026 - Finalizing PCB 3D model
Parts:
- moved D72 23.2 mm to (-1.00, -120.3)
- moved C44 20.4 mm to (283.0, -111.5)
- moved D80 20.2 mm to (281.0, -93.5), turned to 0 degrees
- moved C29 19.1 mm to (283.0, -124.5)
- moved D70 16.8 mm to (231.5, -100.2), turned to 90 degrees
- moved D43 16.6 mm to (280.5, -156.8), turned to -90 degrees
- moved C71 9.01 mm to (280.5, -106.0)
- moved R1 5.72 mm to (291.5, -99.0)
- moved C83 3.54 mm to (292.5, -94.0), turned to -90 degrees
- moved U1 2.24 mm to (297.4, -93.5)
- moved D81 1.69 mm to (279.5, -145.1)
- moved C59 0.50 mm to (17.5, -90.0)

Commit message: 24+26.09.2026 - Plate design
Parts:
- U2: moved to B.Cu
- moved U2 20.8 mm to (303.8, -161.6), turned to 180 degrees
Other:
- board size 314 x 125.5 mm -> 314 x 125 mm

Commit message: # 1 October 2026 - Starting the top case
Parts:
- moved C72 19.3 mm to (-3.00, -77.5), turned to -90 degrees
- moved U2 1.05 mm to (303.8, -160.6)
Other:
- board size 314 x 125 mm -> 313 x 123.5 mm
Changed lines of the file:
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@@
 	(footprint "Capacitor_SMD:C_0805_2012Metric"
 		(layer "F.Cu")
-		(at 16 -74)
+		(at -3 -77.5 -90)
 		(descr "Capacitor SMD 0805 (2012 Metric), square (rectangular) end terminal, IPC-7351 nominal, (Body size source: IPC-SM-782 page 76, https://www.pcb-3d.com/wordpress/wp-content/uploads/ipc-sm-782a_amendment_1_and_2.pdf, https://docs.google.com/spreadsheets/d/1BsfQQcO9C6DZCsRaXUlFlo91Tg2WpOkGARC1WS5S8t0/edit?usp=sharing)")
 		(tags "capacitor")
 		(property "Reference" "C72"
-			(at 0 -1.68 0)
+			(at 0 -1.68 90)
 			(layer "F.SilkS")
 			(effects
@@
 		)
 		(property "Value" "100nF"
-			(at 0 1.68 0)
+			(at 0 1.68 90)
 			(layer "F.Fab")
 			(effects
@@
 		)
 		(property "Datasheet" ""
-			(at 0 0 0)
+			(at 0 0 90)
 			(layer "F.Fab")
 			(hide yes)
@@
 		)
 		(property "Description" "Unpolarized capacitor, small symbol"
-			(at 0 0 0)
+			(at 0 0 90)
 			(layer "F.Fab")
 			(hide yes)
@@
 		)
 		(property "KiLib_Generator" "SMD_2terminal_chip_molded"
-			(at 0 0 0)
+			(at 0 0 90)
 			(layer "F.SilkS")
 			(hide yes)
@@
 		(duplicate_pad_numbers_are_jumpers no)
 		(fp_line
-			(start -0.261252 -0.735)
-			(end 0.261252 -0.735)
+			(start -0.261252 0.735)
+			(end 0.261252 0.735)
 			(stroke
 				(width 0.12)
@@
 		)
 		(fp_line
-			(start -0.261252 0.735)
-			(end 0.261252 0.735)
+			(start -0.261252 -0.735)
+			(end 0.261252 -0.735)
 			(stroke
 				(width 0.12)
@@
 		)
 		(fp_text user "${REFERENCE}"
-			(at 0 0 0)
+			(at 0 0 90)
 			(layer "F.Fab")
 			(effects
@@
 		)
 		(pad "1" smd roundrect
-			(at -0.95 0)
+			(at -0.95 0 270)
 			(size 1 1.45)
 			(layers "F.Cu" "F.Mask" "F.Paste")
@@
 		)
 		(pad "2" smd roundrect
-			(at 0.95 0)
+			(at 0.95 0 270)
 			(size 1 1.45)
 			(layers "F.Cu" "F.Mask" "F.Paste")
@@
 	(footprint "pro_micro_rp2040:pro_micro_rp2040"
 		(layer "B.Cu")
-		(at 303.75 -161.6 180)
+		(at 303.75 -160.55 180)
 		(property "Reference" "U2"
 			(at 8.89 6.46 0)
@@
 	)
 	(gr_line
-		(start -8.5 -195)
-		(end 288.5 -195)
-		(stroke
-			(width 0.05)
-			(type default)
-		)
-		(layer "Edge.Cuts")
-	)
-	(gr_line
-		(start -8.5 -70)
-		(end -8.5 -195)
-		(stroke
-			(width 0.05)
-			(type default)
-		)
-		(layer "Edge.Cuts")
-	)
-	(gr_line
-		(start 288.5 -195)
-		(end 290.5 -194.5)
-		(stroke
-			(width 0.05)
-			(type default)
-		)
-		(layer "Edge.Cuts")
-	)
-	(gr_line
-		(start 290.5 -194.5)
-		(end 299.3 -194.5)
-		(stroke
-			(width 0.05)
-			(type default)
-		)
-		(layer "Edge.Cuts")
-	)
-	(gr_line
-		(start 299.3 -194.5)
-		(end 301.5 -195)
+		(start -7.5 -194)
+		(end 305.5 -194)
 		(stroke
 			(width 0.05)
@@
 	)
 	(gr_line
-		(start 301.5 -195)
-		(end 305.5 -195)
+		(start -7.5 -70.5)
+		(end -7.5 -194)
 		(stroke
 			(width 0.05)
@@
 	)
 	(gr_line
-		(start 305.5 -195)
-		(end 305.5 -70)
+		(start 305.5 -194)
+		(end 305.5 -70.5)
 		(stroke
 			(width 0.05)
@@
 	)
 	(gr_line
-		(start 305.5 -70)
-		(end -8.5 -70)
+		(start 305.5 -70.5)
+		(end -7.5 -70.5)
 		(stroke
 			(width 0.05)
