File: PCB/Crazy-75/Crazy-75.kicad_sch (KiCad schematic)
At the start: 160 parts, among them SW1 SW_Push, SW10 SW_Push, SW11 SW_Push, SW12 SW_Push, SW13 SW_Push, SW14 SW_Push, SW15 SW_Push, SW16 SW_Push, SW17 SW_Push, SW18 SW_Push, SW19 SW_Push, SW2 SW_Push, SW20 SW_Push, SW21 SW_Push, SW22 SW_Push, SW23 SW_Push, SW24 SW_Push, SW25 SW_Push, SW26 SW_Push, SW27 SW_Push, SW28 SW_Push, SW29 SW_Push, SW3 SW_Push, SW30 SW_Push, SW31 SW_Push, SW32 SW_Push, SW33 SW_Push, SW34 SW_Push, SW35 SW_Push, SW36 SW_Push, SW37 SW_Push, SW38 SW_Push, SW39 SW_Push, SW4 SW_Push, SW40 SW_Push, SW41 SW_Push, SW42 SW_Push, SW43 SW_Push, SW44 SW_Push, SW45 SW_Push, SW46 SW_Push, SW47 SW_Push, SW48 SW_Push, SW49 SW_Push, SW5 SW_Push, SW50 SW_Push, SW51 SW_Push, SW52 SW_Push, SW53 SW_Push, SW54 SW_Push, SW55 SW_Push, SW56 SW_Push, SW57 SW_Push, SW58 SW_Push, SW59 SW_Push, SW6 SW_Push, SW60 SW_Push, SW61 SW_Push, SW62 SW_Push, SW63 SW_Push, SW64 SW_Push, SW65 SW_Push, SW66 SW_Push, SW67 SW_Push, SW68 SW_Push, SW69 SW_Push, SW7 SW_Push, SW70 SW_Push, SW71 SW_Push, SW72 SW_Push, SW73 SW_Push, SW74 SW_Push, SW75 SW_Push, SW76 SW_Push, SW77 SW_Push, SW78 SW_Push, SW79 SW_Push, SW8 SW_Push, SW9 SW_Push

Commit message: 06.09.2026 Log
Parts:
- added A1: RaspberryPi_Pico, Module:RaspberryPi_Pico_Common_SMD, symbol MCU_Module:RaspberryPi_Pico
- added C1, C10, C11, C12, C13, C14, C15, C16, C17, C18, C19, C2, C20, C21, C22, C23, C24, C25, C26, C27, C28, C29, C3, C30, C31, C32, C33, C34, C35, C36, C37, C38, C39, C4, C40, C41, C42, C43, C44, C45, C46, C47, C48, C49, C5, C50, C51, C52, C53, C54, C55, C56, C57, C58, C59, C6, C60, C61, C62, C63, C64, C65, C66, C67, C68, C69, C7, C70, C71, C72, C73, C74, C75, C76, C77, C78, C79, C8, C80, C9: 100nF, Capacitor_SMD:C_0805_2012Metric, symbol Device:C_Small
- added D100, D101, D102, D103, D104, D105, D106, D107, D108, D109, D110, D111, D112, D113, D114, D115, D116, D117, D118, D119, D120, D121, D122, D123, D124, D125, D126, D127, D128, D129, D130, D131, D132, D133, D134, D135, D136, D137, D138, D139, D140, D141, D142, D143, D144, D145, D146, D147, D148, D149, D150, D151, D152, D153, D154, D155, D156, D157, D158, D159, D160, D81, D82, D83, D84, D85, D86, D87, D88, D89, D90, D91, D92, D93, D94, D95, D96, D97, D98, D99: SK6812MINI-E, PCM_marbastlib-mx:LED_MX_6028R, symbol PCM_marbastlib-mx:MX_SK6812MINI-E
- added R1: R470, Resistor_THT:R_Axial_DIN0207_L6.3mm_D2.5mm_P10.16mm_Horizontal, symbol Device:R
- added S1: Space, PCM_marbastlib-mx:STAB_MX_P_6.25u, symbol PCM_marbastlib-mx:MX_stab
- added S2, S3: MX_stab, PCM_marbastlib-mx:STAB_MX_P_2.25u, symbol PCM_marbastlib-mx:MX_stab
- added S4: MX_stab, PCM_marbastlib-mx:STAB_MX_P_2u, symbol PCM_marbastlib-mx:MX_stab
- SW1, SW10, SW11, SW12, SW13, SW14, SW15, SW16, SW17, SW18, SW19, SW2, SW20, SW21, SW22, SW23, SW24, SW25, SW26, SW27, SW28, SW29, SW3, SW30, SW31, SW32, SW33, SW34, SW35, SW36, SW37, SW38, SW39, SW4, SW40, SW41, SW42, SW43, SW44, SW45, SW46, SW47, SW48, SW49, SW5, SW50, SW51, SW52, SW53, SW54, SW55, SW56, SW57, SW58, SW59, SW6, SW60, SW61, SW62, SW63, SW64, SW65, SW66, SW67, SW68, SW69, SW7, SW70, SW71, SW72, SW73, SW74, SW75, SW76, SW77, SW78, SW79, SW8, SW9: footprint (none) -> PCM_marbastlib-mx:SW_MX_HS_CPG151101S11_1u; symbol Switch:SW_Push -> PCM_marbastlib-mx:MX_SW_HS_CPG151101S11
- VOL1: renamed from VOL; footprint (none) -> Rotary_Encoder:RotaryEncoder_Alps_EC11E-Switch_Vertical_H20mm
Connections:
- net COL1: now also A1.1 (GPIO0)
- net COL10: now also A1.12 (GPIO9)
- net COL11: now also A1.14 (GPIO10)
- net COL12: now also A1.15 (GPIO11)
- net COL13: now also A1.16 (GPIO12)
- net COL14: now also A1.17 (GPIO13)
- net COL15: now also A1.19 (GPIO14)
- net COL2: now also A1.2 (GPIO1)
- net COL3: now also A1.4 (GPIO2)
- net COL4: now also A1.5 (GPIO3)
- net COL5: now also A1.6 (GPIO4)
- net COL6: now also A1.7 (GPIO5)
- net COL7: now also A1.9 (GPIO6)
- net COL8: now also A1.10 (GPIO7)
- net COL9: now also A1.11 (GPIO8)
- net ROW1: now also A1.20 (GPIO15)
- net ROW2: now also A1.21 (GPIO16)
- net ROW3: now also A1.22 (GPIO17)
- net ROW4: now also A1.24 (GPIO18)
- net ROW5: now also A1.25 (GPIO19)
- net ROW6: now also A1.26 (GPIO20)
- net ENC_A: now reaches VOL1.A
- net ENC_A: now also A1.27 (GPIO21)
- net ENC_B: now reaches VOL1.B
- net ENC_B: now also A1.29 (GPIO22)
- net GND: now reaches VOL1.C
- net GND: now also A1.13 (GND), A1.18 (GND), A1.23 (GND), A1.28 (GND), A1.3 (GND), A1.33 (AGND), A1.38 (GND), A1.8 (GND), C1.2, C10.2, C11.2, C12.2, C13.2, C14.2, C15.2, C16.2, C17.2, C18.2, C19.2, C2.2, C20.2, C21.2, C22.2, C23.2, C24.2, C25.2, C26.2, C27.2, C28.2, C29.2, C3.2, C30.2, C31.2, C32.2, C33.2, C34.2, C35.2, C36.2, C37.2, C38.2, C39.2, C4.2, C40.2, C41.2, C42.2, C43.2, C44.2, C45.2, C46.2, C47.2, C48.2, C49.2, C5.2, C50.2, C51.2, C52.2, C53.2, C54.2, C55.2, C56.2, C57.2, C58.2, C59.2, C6.2, C60.2, C61.2, C62.2, C63.2, C64.2, C65.2, C66.2, C67.2, C68.2, C69.2, C7.2, C70.2, C71.2, C72.2, C73.2, C74.2, C75.2, C76.2, C77.2, C78.2, C79.2, C8.2, C80.2, C9.2, D100.4 (VSS), D101.4 (VSS), D102.4 (VSS), D103.4 (VSS), D104.4 (VSS), D105.4 (VSS), D106.4 (VSS), D107.4 (VSS), D108.4 (VSS), D109.4 (VSS), D110.4 (VSS), D111.4 (VSS), D112.4 (VSS), D113.4 (VSS), D114.4 (VSS), D115.4 (VSS), D116.4 (VSS), D117.4 (VSS), D118.4 (VSS), D119.4 (VSS), D120.4 (VSS), D121.4 (VSS), D122.4 (VSS), D123.4 (VSS), D124.4 (VSS), D125.4 (VSS), D126.4 (VSS), D127.4 (VSS), D128.4 (VSS), D129.4 (VSS), D130.4 (VSS), D131.4 (VSS), D132.4 (VSS), D133.4 (VSS), D134.4 (VSS), D135.4 (VSS), D136.4 (VSS), D137.4 (VSS), D138.4 (VSS), D139.4 (VSS), D140.4 (VSS), D141.4 (VSS), D142.4 (VSS), D143.4 (VSS), D144.4 (VSS), D145.4 (VSS), D146.4 (VSS), D147.4 (VSS), D148.4 (VSS), D149.4 (VSS), D150.4 (VSS), D151.4 (VSS), D152.4 (VSS), D153.4 (VSS), D154.4 (VSS), D155.4 (VSS), D156.4 (VSS), D157.4 (VSS), D158.4 (VSS), D159.4 (VSS), D160.4 (VSS), D81.4 (VSS), D82.4 (VSS), D83.4 (VSS), D84.4 (VSS), D85.4 (VSS), D86.4 (VSS), D87.4 (VSS), D88.4 (VSS), D89.4 (VSS), D90.4 (VSS), D91.4 (VSS), D92.4 (VSS), D93.4 (VSS), D94.4 (VSS), D95.4 (VSS), D96.4 (VSS), D97.4 (VSS), D98.4 (VSS), D99.4 (VSS)
- new net: D103.2 (DOUT), D104.3 (DIN)
- new net: D102.2 (DOUT), D103.3 (DIN)
- new net: D98.2 (DOUT), D99.3 (DIN)
- new net: D97.2 (DOUT), D98.3 (DIN)
- new net: D151.2 (DOUT), D152.3 (DIN)
- new net: D150.2 (DOUT), D151.3 (DIN)
- new net: D138.2 (DOUT), D141.3 (DIN)
- new net: D135.2 (DOUT), D138.3 (DIN)
- new net: D133.2 (DOUT), D136.3 (DIN)
- new net: D130.2 (DOUT), D133.3 (DIN)
- new net: D84.2 (DOUT), D85.3 (DIN)
- new net: D83.2 (DOUT), D84.3 (DIN)
- new net: D87.2 (DOUT), D88.3 (DIN)
- new net: D86.2 (DOUT), D87.3 (DIN)
- new net: D114.2 (DOUT), D115.3 (DIN)
- new net: D113.2 (DOUT), D114.3 (DIN)
- new net: D143.2 (DOUT), D146.3 (DIN)
- new net: D140.2 (DOUT), D143.3 (DIN)
- new net: D123.2 (DOUT), D126.3 (DIN)
- new net: D123.3 (DIN), D149.2 (DOUT)
- new net: D121.2 (DOUT), D124.3 (DIN)
- new net: D120.2 (DOUT), D121.3 (DIN)
- new net: D147.2 (DOUT), D150.3 (DIN)
- new net: D144.2 (DOUT), D147.3 (DIN)
- new net: D88.2 (DOUT), D89.3 (DIN)
- new net: D82.2 (DOUT), D83.3 (DIN)
- new net: D115.2 (DOUT), D116.3 (DIN)
- new net: D131.2 (DOUT), D134.3 (DIN)
- new net: D128.2 (DOUT), D131.3 (DIN)
- new net: D127.2 (DOUT), D130.3 (DIN)
- new net: D124.2 (DOUT), D127.3 (DIN)
- new net: D100.2 (DOUT), D101.3 (DIN)
- new net: D100.3 (DIN), D99.2 (DOUT)
- new net: D93.2 (DOUT), D94.3 (DIN)
- new net: D92.2 (DOUT), D93.3 (DIN)
- new net: D155.2 (DOUT), D156.3 (DIN)
- new net: D154.2 (DOUT), D155.3 (DIN)
- new net: D95.2 (DOUT), D96.3 (DIN)
- new net: D94.2 (DOUT), D95.3 (DIN)
- new net: D152.2 (DOUT), D153.3 (DIN)
- new net: D106.2 (DOUT), D107.3 (DIN)
- new net: D105.2 (DOUT), D106.3 (DIN)
- new net: D104.2 (DOUT), D105.3 (DIN)
- new net: D112.2 (DOUT), D113.3 (DIN)
- new net: D111.2 (DOUT), D112.3 (DIN)
- new net: D107.2 (DOUT), D108.3 (DIN)
- new net: D153.2 (DOUT), D154.3 (DIN)
- new net: D125.2 (DOUT), D128.3 (DIN)
- new net: D122.2 (DOUT), D125.3 (DIN)
- new net: D101.2 (DOUT), D102.3 (DIN)
- new net: D139.2 (DOUT), D142.3 (DIN)
- new net: D136.2 (DOUT), D139.3 (DIN)
- new net: D91.2 (DOUT), D92.3 (DIN)
- new net: D156.2 (DOUT), D157.3 (DIN)
- new net: D116.2 (DOUT), D117.3 (DIN)
- new net: D90.2 (DOUT), D91.3 (DIN)
- new net: D89.2 (DOUT), D90.3 (DIN)
- new net: D126.2 (DOUT), D129.3 (DIN)
- new net: D137.2 (DOUT), D140.3 (DIN)
- new net: D81.2 (DOUT), D82.3 (DIN)
- new net: D158.2 (DOUT), D159.3 (DIN)
- new net: D157.2 (DOUT), D158.3 (DIN)
- new net: D146.2 (DOUT), D149.3 (DIN)
- new net: D159.2 (DOUT), D160.3 (DIN)
- new net: D118.2 (DOUT), D119.3 (DIN)
- new net: D117.2 (DOUT), D118.3 (DIN)
- new net: D119.2 (DOUT), D120.3 (DIN)
- new net: D142.2 (DOUT), D145.3 (DIN)
- new net: D85.2 (DOUT), D86.3 (DIN)
- new net: D141.2 (DOUT), D144.3 (DIN)
- new net: D132.2 (DOUT), D135.3 (DIN)
- new net: D129.2 (DOUT), D132.3 (DIN)
- new net: D81.3 (DIN), R1.2
- new net: D134.2 (DOUT), D137.3 (DIN)
- new net: D122.3 (DIN), D148.2 (DOUT)
- new net: D108.2 (DOUT), D109.3 (DIN)
- new net: D145.2 (DOUT), D148.3 (DIN)
- new net: D96.2 (DOUT), D97.3 (DIN)
- new net: D110.2 (DOUT), D111.3 (DIN)
- new net: D109.2 (DOUT), D110.3 (DIN)
- new net +5V: A1.40 (VBUS), C1.1, C10.1, C11.1, C12.1, C13.1, C14.1, C15.1, C16.1, C17.1, C18.1, C19.1, C2.1, C20.1, C21.1, C22.1, C23.1, C24.1, C25.1, C26.1, C27.1, C28.1, C29.1, C3.1, C30.1, C31.1, C32.1, C33.1, C34.1, C35.1, C36.1, C37.1, C38.1, C39.1, C4.1, C40.1, C41.1, C42.1, C43.1, C44.1, C45.1, C46.1, C47.1, C48.1, C49.1, C5.1, C50.1, C51.1, C52.1, C53.1, C54.1, C55.1, C56.1, C57.1, C58.1, C59.1, C6.1, C60.1, C61.1, C62.1, C63.1, C64.1, C65.1, C66.1, C67.1, C68.1, C69.1, C7.1, C70.1, C71.1, C72.1, C73.1, C74.1, C75.1, C76.1, C77.1, C78.1, C79.1, C8.1, C80.1, C9.1, D100.1 (VDD), D101.1 (VDD), D102.1 (VDD), D103.1 (VDD), D104.1 (VDD), D105.1 (VDD), D106.1 (VDD), D107.1 (VDD), D108.1 (VDD), D109.1 (VDD), D110.1 (VDD), D111.1 (VDD), D112.1 (VDD), D113.1 (VDD), D114.1 (VDD), D115.1 (VDD), D116.1 (VDD), D117.1 (VDD), D118.1 (VDD), D119.1 (VDD), D120.1 (VDD), D121.1 (VDD), D122.1 (VDD), D123.1 (VDD), D124.1 (VDD), D125.1 (VDD), D126.1 (VDD), D127.1 (VDD), D128.1 (VDD), D129.1 (VDD), D130.1 (VDD), D131.1 (VDD), D132.1 (VDD), D133.1 (VDD), D134.1 (VDD), D135.1 (VDD), D136.1 (VDD), D137.1 (VDD), D138.1 (VDD), D139.1 (VDD), D140.1 (VDD), D141.1 (VDD), D142.1 (VDD), D143.1 (VDD), D144.1 (VDD), D145.1 (VDD), D146.1 (VDD), D147.1 (VDD), D148.1 (VDD), D149.1 (VDD), D150.1 (VDD), D151.1 (VDD), D152.1 (VDD), D153.1 (VDD), D154.1 (VDD), D155.1 (VDD), D156.1 (VDD), D157.1 (VDD), D158.1 (VDD), D159.1 (VDD), D160.1 (VDD), D81.1 (VDD), D82.1 (VDD), D83.1 (VDD), D84.1 (VDD), D85.1 (VDD), D86.1 (VDD), D87.1 (VDD), D88.1 (VDD), D89.1 (VDD), D90.1 (VDD), D91.1 (VDD), D92.1 (VDD), D93.1 (VDD), D94.1 (VDD), D95.1 (VDD), D96.1 (VDD), D97.1 (VDD), D98.1 (VDD), D99.1 (VDD)
- new net RBG_DATA: R1.1
- new net RGB_DATA: A1.31 (GPIO26_ADC0)
Other:
- moved on the sheet: SW1, SW10, SW11, SW12, SW13, SW14, SW15, SW16, SW17, SW18, SW19, SW2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

Commit message: Small schematics update
Parts:
- S2: value MX_stab -> Enter
- S3: value MX_stab -> Left Shift
- S4: value MX_stab -> Backspace
Changed lines of the file:
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@@
 			)
 		)
-		(property "Value" "MX_stab"
+		(property "Value" "Enter"
 			(at -180.34 62.1029 0)
 			(show_name no)
@@
 			)
 		)
-		(property "Value" "MX_stab"
+		(property "Value" "Left Shift"
 			(at -180.34 69.7229 0)
 			(show_name no)
@@
 			)
 		)
-		(property "Value" "MX_stab"
+		(property "Value" "Backspace"
 			(at -180.34 77.3429 0)
 			(show_name no)

Commit message: 08.09.2026: PCB work
Parts:
- added C81: 100nF, Capacitor_SMD:C_0805_2012Metric, symbol Device:C_Small
- added D71: 1N4148, Diode_THT:D_DO-35_SOD27_P7.62mm_Horizontal, symbol Diode:1N4148
- added SW71: SW_Push, PCM_marbastlib-mx:SW_MX_HS_CPG151101S11_1u, symbol PCM_marbastlib-mx:MX_SW_HS_CPG151101S11
- added U1: 74AHCT1G125, Package_TO_SOT_SMD:SOT-23-5, symbol 74xGxx:74AHCT1G125
- renumbered D30 to D29, D29 to D30, D33 to D31, D34 to D32, D35 to D33, D36 to D34, D37 to D35, D38 to D36, D39 to D37, D40 to D38, D41 to D39, D42 to D40, D43 to D41, D44 to D42, D45 to D43, D31 to D44, D46 to D45, D47 to D46, D48 to D47, D49 to D48, D50 to D49, D51 to D50, D52 to D51, D53 to D52, D54 to D53, D55 to D54, D56 to D55, D57 to D56, D59 to D57, D32 to D58, D58 to D59, D71 to D72, D72 to D73, D73 to D74, D76 to D75, D74 to D76, D75 to D77, D77 to D79, D79 to D80, D80 to D81, D81 to LED1, D90 to LED10, D91 to LED11, D92 to LED12, D93 to LED13, D94 to LED14, D95 to LED15, D96 to LED16, D97 to LED17, D98 to LED18, D99 to LED19, D82 to LED2, D100 to LED20, D101 to LED21, D102 to LED22, D103 to LED23, D104 to LED24, D105 to LED25, D106 to LED26, D107 to LED27, D108 to LED28, D109 to LED29, D83 to LED3, D110 to LED30, D111 to LED31, D112 to LED32, D113 to LED33, D114 to LED34, D115 to LED35, D116 to LED36, D117 to LED37, D118 to LED38, D119 to LED39, D84 to LED4, D120 to LED40, D121 to LED41, D124 to LED42, D127 to LED43, D130 to LED44, D133 to LED45, D136 to LED46, D139 to LED47, D142 to LED48, D145 to LED49, D85 to LED5, D148 to LED50, D122 to LED51, D125 to LED52, D128 to LED53, D131 to LED54, D134 to LED55, D137 to LED56, D140 to LED57, D143 to LED58, D146 to LED59, D86 to LED6, D149 to LED60, D123 to LED61, D126 to LED62, D129 to LED63, D132 to LED64, D135 to LED65, D138 to LED66, D141 to LED67, D144 to LED68, D147 to LED69, D87 to LED7, D150 to LED70, D151 to LED71, D152 to LED72, D153 to LED73, D154 to LED74, D155 to LED75, D156 to LED76, D157 to LED77, D158 to LED78, D159 to LED79, D88 to LED8, D160 to LED80, D89 to LED9, SW71 to SW72, SW72 to SW73, SW73 to SW74, SW74 to SW75, SW75 to SW76, SW76 to SW77, SW77 to SW78, SW78 to SW79, SW79 to SW80
Connections:
- net +5V: now also C81.1, U1.5 (VCC)
- net COL15: now also SW71.1
- net GND: now also C81.2, U1.1, U1.3 (GND)
- net RGB_DATA: now also U1.2
- net ROW5: now also D71.1 (K)
- net RBG_DATA: no longer names the net of R1.1
- net RBG_DATA: now also U1.4
- new net: D71.2 (A), SW71.2
- no-connect marks 0 -> 8
Other:
- moved on the sheet: A1, D1, D10, D11, D12, D13, D14, D15, D16, D17, D18, D19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

Commit message: 11.09.2026 - PCB design and schematics changes
Parts:
- removed A1: RaspberryPi_Pico, Module:RaspberryPi_Pico_Common_SMD, symbol MCU_Module:RaspberryPi_Pico
- removed C63: 100nF, Capacitor_SMD:C_0805_2012Metric, symbol Device:C_Small
- removed D58: 1N4148, Diode_THT:D_DO-35_SOD27_P7.62mm_Horizontal, symbol Diode:1N4148
- removed LED58: SK6812MINI-E, PCM_marbastlib-mx:LED_MX_6028R, symbol PCM_marbastlib-mx:MX_SK6812MINI-E
- removed SW58: SW_Push, PCM_marbastlib-mx:SW_MX_HS_CPG151101S11_1u, symbol PCM_marbastlib-mx:MX_SW_HS_CPG151101S11
- added C81, C82: 100nF, Capacitor_SMD:C_0805_2012Metric, symbol Device:C_Small
- added LED81, LED82: SK6812MINI-E, PCM_marbastlib-mx:LED_MX_6028R, symbol PCM_marbastlib-mx:MX_SK6812MINI-E
- added U2: (no value), pro_micro_rp2040:pro_micro_rp2040, symbol pro_micro_rp2040:pro_micro_rp2040
- renumbered C44 to C42, C47 to C43, C50 to C44, C53 to C45, C56 to C46, C59 to C47, C62 to C48, C65 to C49, C68 to C50, C42 to C51, C45 to C52, C48 to C53, C51 to C54, C54 to C55, C57 to C56, C60 to C57, C66 to C59, C69 to C60, C43 to C61, C46 to C62, C49 to C63, C52 to C64, C55 to C65, C58 to C66, C61 to C67, C64 to C68, C67 to C69, C81 to C83
Connections:
- net +5V: now also C81.1, C82.1, LED81.1 (VDD), LED82.1 (VDD), U2.5V
- net COL1: now also U2.0 (GP0)
- net COL10: now also U2.9 (GP9)
- net COL11: now also U2.10 (GP10)
- net COL12: now also U2.11 (GP11)
- net COL13: now also U2.12 (GP12)
- net COL14: now also U2.13 (GP13)
- net COL15: now also U2.14 (GP14)
- net COL2: now also U2.1 (GP1)
- net COL3: now also U2.2 (GP2)
- net COL4: now also U2.3 (GP3)
- net COL5: now also U2.4 (GP4)
- net COL6: now also U2.5 (GP5)
- net COL7: now also U2.6 (GP6)
- net COL8: now also U2.7 (GP7)
- net COL9: now also U2.8 (GP8)
- net ENC_A: now also U2.23 (GP23)
- net ENC_B: now also U2.26 (GP26)
- net GND: now also C81.2, C82.2, LED81.4 (VSS), LED82.4 (VSS), U2.GND
- net RGB_DATA: now also U2.27 (GP27)
- net ROW1: now also U2.15 (GP15)
- net ROW2: now also U2.16 (GP16)
- net ROW3: now also U2.18 (GP18)
- net ROW4: now also U2.20 (GP20)
- net ROW5: now also U2.21 (GP21)
- net ROW6: now also U2.22 (GP22)
- net at LED59.3 (DIN): now also LED57.2 (DOUT)
- net at LED80.2 (DOUT): now also LED81.3 (DIN)
- new net: LED81.2 (DOUT), LED82.3 (DIN)
Other:
- moved on the sheet: C1, C10, C11, C12, C13, C14, C15, C16, C17, C18, C19, C2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

Commit message: 13.09.2026 - PCB Mechanical Checks & 3D Validation
Continued working on the physical PCB layout and checking whether the component arrangement would actually work mechanically.
Connections:
- net COL14: now also U2.28 (GP28); no longer U2.13 (GP13)
Changed lines of the file:
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@@
 	)
 	(no_connect
-		(at 157.48 156.21)
+		(at 139.7 184.15)
 	)
 	(no_connect
-		(at 157.48 163.83)
+		(at 157.48 156.21)
 	)
 	(no_connect
@@
 	(wire
 		(pts
-			(xy 139.7 184.15) (xy 139.7 191.77)
-		)
-		(stroke
-			(width 0)
-			(type default)
-		)
-	)
-	(wire
-		(pts
 			(xy 307.34 104.14) (xy 314.96 104.14)
 		)
@@
 		)
 	)
+	(label "COL14"
+		(at 157.48 163.83 0)
+		(effects
+			(font
+				(size 1.27 1.27)
+			)
+			(justify left bottom)
+		)
+	)
 	(label "GND"
 		(at 368.3 60.96 0)
@@
 		(effects
 			(font
-				(size 1.27 1.27)
-			)
-			(justify left bottom)
-		)
-	)
-	(label "COL14"
-		(at 139.7 191.77 90)
-		(effects
-			(font

Commit message: 24.10.2026 - PCB redesign
Parts:
- removed U1: 74AHCT1G125, Package_TO_SOT_SMD:SOT-23-5, symbol 74xGxx:74AHCT1G125
- removed U2: (no value), pro_micro_rp2040:pro_micro_rp2040, symbol pro_micro_rp2040:pro_micro_rp2040
- added C58, C84: 1µF, Capacitor_SMD:C_0805_2012Metric_Pad1.18x1.45mm_HandSolder, symbol Device:C
- added C85: 100nF, Capacitor_SMD:C_0805_2012Metric_Pad1.18x1.45mm_HandSolder, symbol Device:C
- added C86, C87, C88, C89, C90, C91, C92, C93, C94: 100µF, Capacitor_Tantalum_SMD:CP_EIA-7343-31_Kemet-D_HandSolder, symbol Device:C_Polarized
- added J1: USB_C_Receptacle_USB2.0_16P, Connector_USB:USB_C_Receptacle_GCT_USB4085, symbol Connector:USB_C_Receptacle_USB2.0_16P
- added Q1: 2N7002, Package_TO_SOT_SMD:SOT-23_Handsoldering, symbol Transistor_FET:2N7002
- added R2, R3: 5.1k, Resistor_SMD:R_0805_2012Metric_Pad1.20x1.40mm_HandSolder, symbol Device:R
- added R4: 62k, Resistor_SMD:R_0805_2012Metric_Pad1.20x1.40mm_HandSolder, symbol Device:R
- added R5: 110k, Resistor_SMD:R_0805_2012Metric_Pad1.20x1.40mm_HandSolder, symbol Device:R
- added R6, R7, R8, R9: 100k, Resistor_SMD:R_0805_2012Metric_Pad1.20x1.40mm_HandSolder, symbol Device:R
- added SW58: SW_Push, Button_Switch_THT:SW_PUSH_6mm, symbol Switch:SW_Push
- added U1: Frood Rev9 - CUT JP3+JP4, Crazy75:Frood_Rev9_Carrier, symbol Crazy75:Frood_Rev9_CutJP3JP4
- added U3: USBLC6-2SC6, Package_TO_SOT_SMD:SOT-23-6_Handsoldering, symbol Power_Protection:USBLC6-2SC6
- added U4: TPS2553DBVR-MAIN, Package_TO_SOT_SMD:SOT-23-6_Handsoldering, symbol Crazy75:TPS2553DBVR
- added U5: TPS2553DBVR-RGB, Package_TO_SOT_SMD:SOT-23-6_Handsoldering, symbol Crazy75:TPS2553DBVR
- added U7: SN74LV1T125DBV, Package_TO_SOT_SMD:SOT-23-5_HandSoldering, symbol Logic_LevelTranslator:SN74LV1T125DBV
- C1, C10, C11, C12, C13, C14, C15, C16, C17, C18, C19, C2, C20, C21, C22, C23, C24, C25, C26, C27, C28, C29, C3, C30, C31, C32, C33, C34, C35, C36, C37, C38, C39, C4, C40, C41, C42, C43, C44, C45, C46, C47, C48, C49, C5, C50, C51, C52, C53, C54, C55, C56, C57, C59, C6, C60, C61, C62, C63, C64, C65, C66, C67, C68, C69, C7, C70, C71, C72, C73, C74, C75, C76, C77, C78, C79, C8, C80, C81, C82, C83, C9: footprint Capacitor_SMD:C_0805_2012Metric -> Capacitor_SMD:C_0805_2012Metric_Pad1.18x1.45mm_HandSolder
- S2, S3: footprint PCM_marbastlib-mx:STAB_MX_P_2.25u -> PCM_marbastlib-mx:STAB_MX_P_6.25u
- S4: footprint PCM_marbastlib-mx:STAB_MX_P_2u -> PCM_marbastlib-mx:STAB_MX_P_6.25u
Connections:
- net +5V: now also C86.1, C87.1, C88.1, C89.1, C90.1, C91.1, C92.1, C93.1, C94.1, U5.6 (OUT); no longer C83.1
- net COL1: now also U1.2 (GPIO0)
- net COL10: now also U1.13 (GPIO9)
- net COL11: now also U1.4 (GP10)
- net COL12: now also U1.5 (GP11)
- net COL13: now also U1.14 (GPIO12)
- net COL14: now also U1.25 (GPIO28)
- net COL15: now also U1.16 (GPIO14)
- net COL2: now also U1.3 (GPIO1)
- net COL3: now also U1.6 (GPIO2)
- net COL4: now also U1.7 (GPIO3)
- net COL5: now also U1.8 (GPIO4)
- net COL6: now also U1.9 (GPIO5)
- net COL7: now also U1.10 (GPIO6)
- net COL8: now also U1.11 (GPIO7)
- net COL9: now also U1.12 (GPIO8)
- net ENC_A: now also U1.20 (GPIO23)
- net ENC_B: now also U1.23 (GPIO26)
- net GND: now also C58.2, C84.2, C85.2, C86.2, C87.2, C88.2, C89.2, C90.2, C91.2, C92.2, C93.2, C94.2, J1.A1 (GND), J1.A12 (GND), J1.B1 (GND), J1.B12 (GND), J1.SH (SHIELD), Q1.2 (S), R2.2, R3.2, R4.1, R5.1, R6.2, R7.2, R8.1, SW58.2, U1.29 (GND), U3.2 (GND), U4.2 (GND), U5.2 (GND), U7.3 (GND)
- net RGB_DATA: now also R7.1, U1.24 (GPIO27), U7.2 (A)
- net ROW1: now also U1.17 (GPIO15)
- net ROW2: now also U1.18 (GPIO16)
- net ROW3: now also U1.15 (GPIO13)
- net ROW4: now also U1.21 (GPIO20)
- net ROW5: now also U1.19 (GPIO21)
- net ROW6: now also U1.22 (GPIO22)
- net at R1.1: now also U7.4 (Y)
- net at LED1.3 (DIN), R1.2: now also R8.2
- new net: J1.B5 (CC2), R3.1
- new net: R4.2, U4.5 (ILIM)
- new net: SW58.1, U1.28 (RST)
- new net: R5.2, U5.5 (ILIM)
- new net: J1.A5 (CC1), R2.1
- new net +5V_SYS: C83.1, C84.1, C85.1, R9.2, U1.30 (RAW), U4.6 (OUT), U5.1 (IN), U7.5 (VCC)
- new net CONN_DM: J1.A7 (D-), J1.B7 (D-), U3.3 (I/O2)
- new net CONN_DP: J1.A6 (D+), J1.B6 (D+), U3.1 (I/O1)
- new net RGB_EN: Q1.1 (G), R6.1, U1.26 (GPIO29), U5.3 (EN)
- new net RGB_OE_N: Q1.3 (D), R9.1, U7.1 (~{OE})
- new net USB_DM: U1.31 (USB_D-), U3.4 (I/O2)
- new net USB_DP: U1.1 (USB_D+), U3.6 (I/O1)
- new net VBUS_USB: C58.1, J1.A4 (VBUS), J1.A9 (VBUS), J1.B4 (VBUS), J1.B9 (VBUS), U3.5 (VBUS), U4.1 (IN), U4.3 (EN)
- no-connect marks 8 -> 6
